File: pcb/bakeneko-60-pcb.sch (KiCad schematic (older format))
At the start: 18 parts, among them J1 JST SH 4-pin, J2 AVR-ISP-6, SW1 Reset, U1 SRV05-4, U2 ATmega32U4-AU, Y1 16MHz

Commit message: Update bakeneko-60-pcb.sch
Other:
- moved on the sheet: C1, C2, C3, C4, C5, C6, C7, F1, J1, J2, R1, R2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

Commit message: Update PCB
Parts:
- J2: footprint random-keyboard-parts:Reset_Pretty -> bakeneko:ISP
Changed lines of the file:
@@
 F 0 "J2" H 1971 1746 50  0000 R CNN
 F 1 "AVR-ISP-6" H 1971 1655 50  0000 R CNN
-F 2 "random-keyboard-parts:Reset_Pretty" V 2050 1700 50  0001 C CNN
+F 2 "bakeneko:ISP" V 2050 1700 50  0001 C CNN
 F 3 " ~" H 1025 1100 50  0001 C CNN
 	1    2300 1650
